File: progetto-eagle/PCB2D-amplificatore-audio.brd (EAGLE design)
At the start: 87.6 x 72.1 mm, 26 parts, among them J1 AUDIO_JACK_TRS_0.25"_PTH_RA, J2 AUDIO_JACK_TRS_0.25"_PTH_RA, J3 DCJ0202, U1 LM386_SOIC, U2 OPA1678IDGKR

Commit message: finito
completato tutto
Parts:
- R3, R4: value 100k -> 10k
Changed lines of the file:
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@@
 <attribute name="VALUE" x="22.1234" y="40.2844" size="1.27" layer="27" rot="R270"/>
 </element>
-<element name="R3" library="rcl" library_urn="urn:adsk.eagle:library:334" package="R0603" package3d_urn="urn:adsk.eagle:package:23555/3" value="100k" base_value="100k" x="17.78" y="56.0832" smashed="yes">
+<element name="R3" library="rcl" library_urn="urn:adsk.eagle:library:334" package="R0603" package3d_urn="urn:adsk.eagle:package:23555/3" value="10k" base_value="10k" x="17.78" y="56.0832" smashed="yes">
 <attribute name="NAME" x="16.4592" y="57.404" size="1.27" layer="25"/>
 <attribute name="POPULARITY" value="77" x="54.61" y="7.8232" size="1.778" layer="27" display="off"/>
@@
 <attribute name="VALUE" x="12.192" y="55.7022" size="1.27" layer="27"/>
 </element>
-<element name="R4" library="rcl" library_urn="urn:adsk.eagle:library:334" package="R0603" package3d_urn="urn:adsk.eagle:package:23555/3" value="100k" base_value="100k" x="28.4734" y="59.7916" smashed="yes" rot="R180">
+<element name="R4" library="rcl" library_urn="urn:adsk.eagle:library:334" package="R0603" package3d_urn="urn:adsk.eagle:package:23555/3" value="10k" base_value="10k" x="28.4734" y="59.7916" smashed="yes" rot="R180">
 <attribute name="NAME" x="30.48" y="62.357" size="1.27" layer="25" rot="R180"/>
 <attribute name="POPULARITY" value="77" x="-14.7066" y="108.0516" size="1.778" layer="27" rot="R180" display="off"/>
